File: pcb/ssd1327.kicad_pcb (KiCad board)
At the start: 2 copper layers, 0 parts

Commit message: SSD1327 PCB routing
Parts:
- added C1: 1uF, Capacitor_SMD:C_0603_1608Metric, F.Cu at (40.6, 52.6)
- added C10: 22uF (25V), Capacitor_SMD:C_0805_2012Metric, F.Cu at (58.2, 49.5)
- added C11: 10uF (25V), Capacitor_SMD:C_0603_1608Metric, F.Cu at (63.0, 49.6)
- added C12: 0.1uF (25V), Capacitor_SMD:C_0603_1608Metric, F.Cu at (61.5, 49.6)
- added C2: 4.7uF (25V), Capacitor_SMD:C_0603_1608Metric, F.Cu at (63.0, 52.6)
- added C3: 10uF, Capacitor_SMD:C_0603_1608Metric, F.Cu at (66.8, 31.7)
- added C4: 0.1uF, Capacitor_SMD:C_0603_1608Metric, F.Cu at (53.2, 31.2)
- added C5: 1uF, Capacitor_SMD:C_0603_1608Metric, F.Cu at (52.8, 39.8)
- added C6: 2.2uF, Capacitor_SMD:C_0603_1608Metric, F.Cu at (52.8, 41.3)
- added C7: 10uF, Capacitor_SMD:C_0603_1608Metric, F.Cu at (53.2, 32.7)
- added C8: 0.1uF, Capacitor_SMD:C_0603_1608Metric, F.Cu at (53.2, 34.2)
- added C9: 22uF, Capacitor_SMD:C_0805_2012Metric, F.Cu at (62.5, 43.3)
- added D1: SS34, Diode_SMD:D_SMA, F.Cu at (58.0, 43.3)
- added J1: Display Connector Input, Connector_Molex:Molex_PicoBlade_53261-1071_1x10-1MP_P1.25mm_Horizontal, F.Cu at (67.5, 45.2)
- added J2: SSD1327 16-Pin Connector, Display_FPC:ssd1327, F.Cu at (50.2, 52.2)
- added J3: USB_C_Receptacle_USB2.0_16P, Connector_USB:USB_C_Receptacle_HCTL_HC-TYPE-C-16P-01A, F.Cu at (60.0, 33.6)
- added L1: 22uH (or 10uH), Inductor_SMD:L_0603_1608Metric, F.Cu at (54.8, 45.8)
- added R1: 10k, Resistor_SMD:R_0603_1608Metric, F.Cu at (61.7, 40.0)
- added R10: 10k, Resistor_SMD:R_0603_1608Metric, F.Cu at (62.3, 47.3)
- added R2: 1M, Resistor_SMD:R_0603_1608Metric, F.Cu at (39.1, 52.6)
- added R3: 5.1k, Resistor_SMD:R_0603_1608Metric, F.Cu at (66.8, 33.2)
- added R4: 5.1k, Resistor_SMD:R_0603_1608Metric, F.Cu at (66.8, 34.7)
- added R5: 22R, Resistor_SMD:R_0603_1608Metric, F.Cu at (60.2, 40.0)
- added R6: 22R, Resistor_SMD:R_0603_1608Metric, F.Cu at (58.7, 40.0)
- added R7: 10k, Resistor_SMD:R_0603_1608Metric, F.Cu at (52.8, 42.8)
- added R8: 100k, Resistor_SMD:R_0603_1608Metric, F.Cu at (62.3, 45.8)
- added R9: 190k (or 200k), Resistor_SMD:R_0603_1608Metric, F.Cu at (55.6, 48.1)
- added U1: AP2112K-3.3, Package_TO_SOT_SMD:SOT-23-5, F.Cu at (52.9, 37.0)
- added U2: ESP32-S3-WROOM-1, RF_Module:ESP32-S3-WROOM-1, F.Cu at (36.8, 40.0)
- added U3: MT3608, Package_TO_SOT_SMD:SOT-23-6, F.Cu at (58.4, 46.8)
Routing:
- net +5V: track 0.00 -> 68.9 mm, vias 0 -> 6
- net /ESP32 for SSD1327/3V3: track 0.00 -> 66.5 mm, vias 0 -> 5
- net /ESP32 for SSD1327/CLK: track 0.00 -> 31.2 mm, vias 0 -> 2
- net /ESP32 for SSD1327/MOSI: track 0.00 -> 30.1 mm, vias 0 -> 2
- net /ESP32 for SSD1327/GPIO39: track 0.00 -> 29.1 mm, vias 0 -> 2
- net /ESP32 for SSD1327/GPIO1: track 0.00 -> 28.8 mm, vias 0 -> 2
- net /ESP32 for SSD1327/MISO: track 0.00 -> 28.7 mm, vias 0 -> 2
- net Net-(U2-EN): track 0.00 -> 27.2 mm, vias 0 -> 2
- net /ESP32 for SSD1327/GPIO13: track 0.00 -> 24.3 mm, vias 0 -> 2
- net Net-(U2-USB_D-): track 0.00 -> 21.0 mm
- net /MT3608 for SSD1327/12V: track 0.00 -> 20.2 mm, vias 0 -> 2
- net /ESP32 for SSD1327/GPIO14: track 0.00 -> 19.7 mm, vias 0 -> 2
- net /ESP32 for SSD1327/GPIO21: track 0.00 -> 19.1 mm, vias 0 -> 2
- net GND: track 0.00 -> 16.3 mm, vias 0 -> 7
- net Net-(U2-USB_D+): track 0.00 -> 16.2 mm
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- added copper zone on B.Cu, net GND
- added copper zone on F.Cu, net GND
Other:
- board outline added: 40 x 25 mm
- board text added: "Jonathan Ho 2026-03-12"
- board text added: "SSD1327 Display Adapter"
