File: pcb/ssd1327.kicad_pcb (KiCad board)
At the start: 2 copper layers, 40 x 25 mm, 30 parts, among them J1 Display Connector Input, J2 SSD1327 16-Pin Connector, J3 USB_C_Receptacle_USB2.0_16P, U1 AP2112K-3.3, U2 ESP32-S3-WROOM-1, U3 MT3608

Commit message: Master board PCB routing
Parts:
- C10: value 22uF (25V) -> 22uF
- C11: value 10uF (25V) -> 10uF
- C12: value 0.1uF (25V) -> 0.1uF
- C2: value 4.7uF (25V) -> 4.7uF
- L1: value 22uH (or 10uH) -> 10uH
- R9: value 190k (or 200k) -> 200k
Changed lines of the file:
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@@
 			)
 		)
-		(property "Value" "190k (or 200k)"
+		(property "Value" "200k"
 			(at 48.1 -55.6 0)
 			(layer "F.Fab")
@@
 			)
 		)
-		(property "Value" "10uF (25V)"
+		(property "Value" "10uF"
 			(at 49.6 -63 0)
 			(layer "F.Fab")
@@
 			)
 		)
-		(property "Value" "0.1uF (25V)"
+		(property "Value" "0.1uF"
 			(at 49.6 -61.5 0)
 			(layer "F.Fab")
@@
 			)
 		)
-		(property "Value" "4.7uF (25V)"
+		(property "Value" "4.7uF"
 			(at -52.6 63 0)
 			(layer "F.Fab")
@@
 			)
 		)
-		(property "Value" "22uH (or 10uH)"
+		(property "Value" "10uH"
 			(at -54.8 -45.8 0)
 			(layer "F.Fab")
@@
 			)
 		)
-		(property "Value" "22uF (25V)"
+		(property "Value" "22uF"
 			(at 58.2 49.5 0)
 			(layer "F.Fab")
@@
 	)
 	(gr_text "SSD1327 Display Adapter"
-		(at 68 32 0)
+		(at 32 32 0)
 		(layer "B.SilkS")
 		(effects
@@
 				(bold yes)
 			)
-			(justify left top mirror)
+			(justify right top mirror)
 		)
 	)
 	(gr_text "Jonathan Ho\n2026-03-12"
-		(at 68 34 0)
+		(at 32 34 0)
 		(layer "B.SilkS")
 		(effects
@@
 				(thickness 0.125)
 			)
-			(justify left top mirror)
+			(justify right top mirror)
 		)
 	)
