File: pcb/master.kicad_sch (KiCad schematic)
At the start: 15 parts, among them J1 Micro_SD_Card, J2 Display Connector Output, J3 Display Connector Output, J4 Display Connector Output

Commit message: Master board PCB routing
Parts:
- removed J1: Micro_SD_Card, Connector_Card:microSD_HC_Molex_47219-2001, symbol Connector:Micro_SD_Card
- added J1: Micro_SD_Card_Det2, Connector_Card:microSD_HC_Hirose_DM3AT-SF-PEJM5, symbol Connector:Micro_SD_Card_Det2
Connections:
- net CLK: now also J1.5 (CLK)
- net GND: now also J1.11 (SHIELD), J1.6 (VSS)
- net MISO: now also J1.7 (DAT0)
- net MOSI: now also J1.3 (CMD)
- net Master ESP32/3V3: now also J1.4 (VDD)
- net Master ESP32/GPIO12: now also J1.2 (DAT3/CD)
- net at R6.2: now also J1.1 (DAT2)
- net at R1.2: now also J1.8 (DAT1)
Changed lines of the file:
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@@
+	)
+	(symbol
+		(lib_id "Connector:Micro_SD_Card_Det2")
+		(at 90.17 48.26 0)
+		(unit 1)
+		(exclude_from_sim no)
+		(in_bom yes)
+		(on_board yes)
+		(dnp no)
+		(fields_autoplaced yes)
+		(property "Reference" "J1"
+			(at 90.805 26.67 0)
+			(effects
+				(font
+					(size 1.27 1.27)
+				)
+			)
+		)
+		(property "Value" "Micro_SD_Card_Det2"
+			(at 90.805 29.21 0)
+			(effects
+				(font
+					(size 1.27 1.27)
+				)
+			)
+		)
+		(property "Footprint" "Connector_Card:microSD_HC_Hirose_DM3AT-SF-PEJM5"
+			(at 142.24 30.48 0)
+			(effects
+				(font
+					(size 1.27 1.27)
+				)
+				(hide yes)
+			)
+		)
+		(property "Datasheet" "https://www.hirose.com/en/product/document?clcode=&productname=&series=DM3&documenttype=Catalog&lang=en&documentid=D49662_en"
+			(at 92.71 45.72 0)
+			(effects
+				(font
+					(size 1.27 1.27)
+				)
+				(hide yes)
+			)
+		)
+		(property "Description" "Micro SD Card Socket with two card detection pins"
+			(at 90.17 48.26 0)
+			(effects
+				(font
+					(size 1.27 1.27)
+				)
+				(hide yes)
+			)
+		)
+		(pin "8"
+		)
+		(pin "4"
+		)
+		(pin "3"
+		)
+		(pin "6"
+		)
+		(pin "2"
+		)
+		(pin "1"
+		)
+		(pin "7"
+		)
+		(pin "10"
+		)
+		(pin "11"
+		)
+		(pin "5"
+		)
+		(pin "9"
+		)
+		(instances
+			(project ""
+				(path "/ef60a031-d3da-483e-916d-caebb8513ab6"
+					(reference "J1")
+					(unit 1)
+				)
+			)
+		)
 	)
 	(symbol
@@
 					(unit 1)
 				)
-			)
-		)
-	)
-	(symbol
-		(lib_id "Connector:Micro_SD_Card")
-		(at 90.17 45.72 0)
-		(unit 1)
-		(exclude_from_sim no)
-		(in_bom yes)
-		(on_board yes)
-		(dnp no)
-		(fields_autoplaced yes)
-		(property "Reference" "J1"
-			(at 90.805 26.67 0)
-			(effects
-				(font
-					(size 1.27 1.27)
-				)
-			)
-		)
-		(property "Value" "Micro_SD_Card"
-			(at 90.805 29.21 0)
-			(effects
-				(font
-					(size 1.27 1.27)
-				)
-			)
-		)
-		(property "Footprint" "Connector_Card:microSD_HC_Molex_47219-2001"
-			(at 119.38 38.1 0)
-			(effects
-				(font
-					(size 1.27 1.27)
-				)
-				(hide yes)
-			)
-		)
-		(property "Datasheet" "https://www.we-online.com/components/products/datasheet/693072010801.pdf"
-			(at 90.17 45.72 0)
-			(effects
-				(font
-					(size 1.27 1.27)
-				)
-				(hide yes)
-			)
-		)
-		(property "Description" "Micro SD Card Socket"
-			(at 90.17 45.72 0)
-			(effects
-				(font
-					(size 1.27 1.27)
-				)
-				(hide yes)
-			)
-		)
-		(pin "2"
-		)
-		(pin "1"
-		)
-		(pin "3"
-		)
-		(pin "4"
-		)
-		(pin "5"
-		)
-		(pin "6"
-		)
-		(pin "7"
-		)
-		(pin "9"
-		)
-		(pin "8"
-		)
-		(instances
-			(project ""
-				(path "/ef60a031-d3da-483e-916d-caebb8513ab6"
-					(reference "J1")
-					(unit 1)
-				)
