File: pcb/master.kicad_sch (KiCad schematic)
At the start: 15 parts, among them J1 Micro_SD_Card_Det2, J2 Display Connector Output, J3 Display Connector Output, J4 Display Connector Output

Commit message: Update project version and references
Parts:
- J2, J3, J4: symbol Data Connector:Display_Connector_Output -> Data_Connector:Display_Connector_Output
Connections:
- net GND: now also J1.SH (SHIELD); no longer J1.11 (SHIELD)
