File: pcb/esp32.kicad_sch (KiCad schematic)
At the start: 14 parts, among them J5 USB_C_Receptacle_USB2.0_16P, U1 AP2112K-3.3, U2 ESP32-S3-WROOM-1

Commit message: Update project version and references
Connections:
- net GND: now also J5.SH (SHIELD); no longer J5.S1 (SHIELD)
