File: pcb/mt3608.kicad_sch (KiCad schematic)
At the start: 10 parts, among them U3 MT3608

Commit message: Update project version and references
Parts:
- renumbered C11 to C10, C12 to C11, C13 to C12, C10 to C9, D3 to D1, R11 to R10, R9 to R8, R10 to R9
