File: pcb/ssd1322.kicad_pcb (KiCad board)
At the start: 2 copper layers, 40 x 25 mm, 34 parts, among them J1 Display Connector Input, J2 SSD1322 30-Pin Connector, J3 USB_C_Receptacle_USB2.0_16P, U1 AP2112K-3.3, U2 ESP32-S3-WROOM-1, U3 MT3608

Commit message: Update project version and references
Parts:
- J2: footprint Display_FPC:ssd1322 -> Display_FPC:30-pin
