File: pcb/ssd1322.kicad_sch (KiCad schematic)
At the start: 10 parts, among them J1 Display Connector Input, J2 SSD1322 30-Pin Connector

Commit message: Update project version and references
Parts:
- D1, D2: footprint Diode_SMD:D_SOD-123 -> Diode_THT:D_DO-35_SOD27_P7.62mm_Horizontal
- J1: symbol Data Connector:Display_Connector_Input -> Data_Connector:Display_Connector_Input
- J2: footprint Display_FPC:ssd1322 -> Display_FPC:30-pin; symbol SSD1322:SSD1322_30-Pin_Connector -> OLED_Driver:SSD1322_30-Pin_Connector
