File: pcb/ssd1327.kicad_sch (KiCad schematic)
At the start: 6 parts, among them J1 Display Connector Input, J2 SSD1327 16-Pin Connector

Commit message: Update project version and references
Parts:
- J1: symbol Data Connector:Display_Connector_Input -> Data_Connector:Display_Connector_Input
- J2: footprint Display_FPC:ssd1327 -> Display_FPC:16-pin; symbol SSD1327:SSD1327_16-Pin_Connector -> OLED_Driver:SSD1327_16-Pin_Connector
